File: oc-v1/oc-kicad/oc/oc.kicad_sch (KiCad schematic)
At the start: 16 parts, among them U1 JOYSTICKPTH, U2 JOYSTICKPTH, X1 SW_Push, Y1 SW_Push

Commit message: WIP
Parts:
- added D1, D2, D3, D4: (no value), LED_THT:LED_D5.0mm-4_RGB_Wide_Pins, symbol liam_custom:WS2812_5mm
- added SW14, SW15: SW_Push, Button_Switch_THT:SW_PUSH-12mm, symbol Switch:SW_Push
- added U1: (no value), Module:Maple_Mini, symbol liam_custom:MUX_Breakout_CD74HC4067
- renumbered U1 to J1, U2 to J2, LEFT to SW1, RB1 to SW10, Y1 to SW11, A2 to SW12, B1 to SW13, LB1 to SW2, UP to SW3, DOWN to SW4, RIGHT to SW5, SELECT1 to SW6, HOME1 to SW7, START1 to SW8, X1 to SW9
Connections:
- net +3V3: now also A1.36 (3V3), U1.23 (VCC)
- net BTN_A: now also A1.6 (GPIO4)
- net BTN_B: now also A1.7 (GPIO5)
- net BTN_DOWN: now also A1.20 (GPIO15)
- net BTN_HOME: now also A1.25 (GPIO19)
- net BTN_LB: now also A1.21 (GPIO16)
- net BTN_LEFT: now also A1.16 (GPIO12)
- net BTN_RB: now also A1.22 (GPIO17)
- net BTN_RIGHT: now also A1.19 (GPIO14)
- net BTN_SEL: now also A1.24 (GPIO18)
- net BTN_START: now also A1.26 (GPIO20)
- net BTN_UP: now also A1.17 (GPIO13)
- net BTN_X: now also A1.4 (GPIO2)
- net BTN_Y: now also A1.5 (GPIO3)
- net GND: now also A1.33 (AGND), D1.2 (GND), D2.2 (GND), D3.2 (GND), D4.2 (GND), SW14.1, SW15.1, U1.18 (S3), U1.19 (S2), U1.22 (EN), U1.24 (GND)
- net JL_SEL: now also A1.11 (GPIO8)
- net JL_X: now also U1.1 (C0)
- net JL_Y: now also U1.2 (C1)
- net JR_SEL: now also A1.12 (GPIO9)
- net JR_X: now also U1.3 (C2)
- net JR_Y: now also U1.4 (C3)
- net AMUX_S1: now reaches A1.10 (GPIO7)
- net AMUX_S1: now also U1.20 (S1)
- net BTN_C: now reaches A1.14 (GPIO10)
- net BTN_C: now also A1.27 (GPIO21), SW14.2
- net BTN_Z: now reaches A1.15 (GPIO11)
- net BTN_Z: now also A1.29 (GPIO22), SW15.2
- net AMUX_SIG: now reaches A1.31 (GPIO26_ADC0)
- net AMUX_SIG: now also U1.17 (SIG)
- net RGB_DIN: now reaches A1.32 (GPIO27_ADC1)
- net RGB_DIN: now also D1.1 (DIN)
- net +5V: now reaches A1.40 (VBUS)
- net +5V: now also D1.3 (VCC), D2.3 (VCC), D3.3 (VCC), D4.3 (VCC)
- net AMUX_S0: now reaches A1.9 (GPIO6)
- net AMUX_S0: now also U1.21 (S0)
- new net: D1.4 (OUTPUT), D2.1 (DIN)
- new net: D2.4 (OUTPUT), D3.1 (DIN)
- new net: D3.4 (OUTPUT), D4.1 (DIN)
- no-connect marks 0 -> 22
Other:
- company: (none) -> Liam Swift
- title: (none) -> OpenController V1
- moved on the sheet: A1, SW1, SW10, SW11, SW12, SW13, SW2, SW3, SW4, SW5, SW6, SW7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

Commit message: Add MUX breakout
Parts:
- A1: footprint Module:RaspberryPi_Pico_SMD_HandSolder -> Module:RaspberryPi_Pico_Common_THT
- U1: footprint Module:Maple_Mini -> mux_breakout:MuxBreakout
Other:
- company: Liam Swift -> Liam Dobbelaere
Changed lines of the file:
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@@
 		(date "2026-09-27")
 		(rev "1")
-		(company "Liam Swift")
+		(company "Liam Dobbelaere")
 	)
 	(no_connect
@@
 			)
 		)
-		(property "Footprint" "Module:Maple_Mini"
+		(property "Footprint" "mux_breakout:MuxBreakout"
 			(at 43.18 168.91 0)
 			(hide yes)
@@
 			)
 		)
-		(property "Footprint" "Module:RaspberryPi_Pico_SMD_HandSolder"
+		(property "Footprint" "Module:RaspberryPi_Pico_Common_THT"
 			(at 50.8 109.22 0)
 			(hide yes)

Commit message: Update
Parts:
- removed J1, J2: JOYSTICKPTH, adafruit_joystick_v2:JOYSTICK, symbol joystick-eagle-import:JOYSTICKPTH
- added J1, J2: (no value), adafruit_joystick_v2:JOYSTICK, symbol Adafruit_joy_library:JOYSTICKPTH
Connections:
- net +3V3: now also D1.3 (VCC), D2.3 (VCC), D3.3 (VCC), D4.3 (VCC), J1.H1 (H+), J1.V1 (V+), J2.H1 (H+), J2.V1 (V+)
- net +5V: no longer D1.3 (VCC), D2.3 (VCC), D3.3 (VCC), D4.3 (VCC)
- net GND: now also J1.B2A (SEL-), J1.H3 (H-), J1.V3 (V-), J2.B2A (SEL-), J2.H3 (H-), J2.V3 (V-)
- net JL_SEL: now also J1.B1A (SEL+)
- net JL_X: now also J1.H2 (H)
- net JL_Y: now also J1.V2 (V)
- net JR_SEL: now also J2.B1A (SEL+)
- net JR_X: now also J2.H2 (H)
- net JR_Y: now also J2.V2 (V)

Commit message: PCB WIP
Parts:
- SW1, SW11, SW12, SW13, SW14, SW15, SW3, SW4, SW5, SW6, SW7, SW8, SW9: footprint Button_Switch_THT:SW_PUSH-12mm -> Button_Switch_THT:SW_PUSH_6mm
Changed lines of the file:
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@@
 			)
 		)
-		(property "Footprint" "Button_Switch_THT:SW_PUSH-12mm"
+		(property "Footprint" "Button_Switch_THT:SW_PUSH_6mm"
 			(at 168.91 33.02 0)
 			(hide yes)
@@
 			)
 		)
-		(property "Footprint" "Button_Switch_THT:SW_PUSH-12mm"
+		(property "Footprint" "Button_Switch_THT:SW_PUSH_6mm"
 			(at 101.6 90.17 0)
 			(hide yes)
@@
 			)
 		)
-		(property "Footprint" "Button_Switch_THT:SW_PUSH-12mm"
+		(property "Footprint" "Button_Switch_THT:SW_PUSH_6mm"
 			(at 111.76 77.47 0)
 			(hide yes)
@@
 			)
 		)
-		(property "Footprint" "Button_Switch_THT:SW_PUSH-12mm"
+		(property "Footprint" "Button_Switch_THT:SW_PUSH_6mm"
 			(at 189.23 60.96 0)
 			(hide yes)
@@
 			)
 		)
-		(property "Footprint" "Button_Switch_THT:SW_PUSH-12mm"
+		(property "Footprint" "Button_Switch_THT:SW_PUSH_6mm"
 			(at 232.41 73.66 0)
 			(hide yes)
@@
 			)
 		)
-		(property "Footprint" "Button_Switch_THT:SW_PUSH-12mm"
+		(property "Footprint" "Button_Switch_THT:SW_PUSH_6mm"
 			(at 217.17 86.36 0)
 			(hide yes)
@@
 			)
 		)
-		(property "Footprint" "Button_Switch_THT:SW_PUSH-12mm"
+		(property "Footprint" "Button_Switch_THT:SW_PUSH_6mm"
 			(at 199.39 48.26 0)
 			(hide yes)
@@
 			)
 		)
-		(property "Footprint" "Button_Switch_THT:SW_PUSH-12mm"
+		(property "Footprint" "Button_Switch_THT:SW_PUSH_6mm"
 			(at 199.39 72.39 0)
 			(hide yes)
@@
 			)
 		)
-		(property "Footprint" "Button_Switch_THT:SW_PUSH-12mm"
+		(property "Footprint" "Button_Switch_THT:SW_PUSH_6mm"
 			(at 111.76 101.6 0)
 			(hide yes)
@@
 			)
 		)
-		(property "Footprint" "Button_Switch_THT:SW_PUSH-12mm"
+		(property "Footprint" "Button_Switch_THT:SW_PUSH_6mm"
 			(at 146.05 33.02 0)
 			(hide yes)
@@
 			)
 		)
-		(property "Footprint" "Button_Switch_THT:SW_PUSH-12mm"
+		(property "Footprint" "Button_Switch_THT:SW_PUSH_6mm"
 			(at 121.92 90.17 0)
 			(hide yes)
@@
 			)
 		)
-		(property "Footprint" "Button_Switch_THT:SW_PUSH-12mm"
+		(property "Footprint" "Button_Switch_THT:SW_PUSH_6mm"
 			(at 124.46 33.02 0)
 			(hide yes)
@@
 			)
 		)
-		(property "Footprint" "Button_Switch_THT:SW_PUSH-12mm"
+		(property "Footprint" "Button_Switch_THT:SW_PUSH_6mm"
 			(at 209.55 60.96 0)
 			(hide yes)
