File: oc-v1/oc-kicad/oc/oc.kicad_pcb (KiCad board)
At the start: 2 copper layers, 1 part

Commit message: PCB WIP
Parts:
- added D1: ~, LED_THT:LED_D5.0mm-4_RGB_Wide_Pins, F.Cu at (254.3, 58.8)
- added D2: ~, LED_THT:LED_D5.0mm-4_RGB_Wide_Pins, F.Cu at (254.3, 66.3)
- added D3: ~, LED_THT:LED_D5.0mm-4_RGB_Wide_Pins, F.Cu at (254.3, 73.9)
- added D4: ~, LED_THT:LED_D5.0mm-4_RGB_Wide_Pins, F.Cu at (254.3, 81.4)
- added J1: ~, adafruit_joystick_v2:JOYSTICK, F.Cu at (0.00, 0.00)
- added J2: ~, adafruit_joystick_v2:JOYSTICK, F.Cu at (62.0, 28.0)
- added SW1: SW_Push, Button_Switch_THT:SW_PUSH_6mm, F.Cu at (3.25, 25.5)
- added SW10: SW_Push, Button_Switch_THT:SW_PUSH-12mm, F.Cu at (190.3, 106.9)
- added SW11: SW_Push, Button_Switch_THT:SW_PUSH_6mm, F.Cu at (74.8, -12.2)
- added SW12: SW_Push, Button_Switch_THT:SW_PUSH_6mm, F.Cu at (74.8, 7.75)
- added SW13: SW_Push, Button_Switch_THT:SW_PUSH_6mm, F.Cu at (85.8, -2.25)
- added SW14: SW_Push, Button_Switch_THT:SW_PUSH_6mm, F.Cu at (83.8, 25.8)
- added SW15: SW_Push, Button_Switch_THT:SW_PUSH_6mm, F.Cu at (97.8, 15.8)
- added SW2: SW_Push, Button_Switch_THT:SW_PUSH-12mm, F.Cu at (173.6, 75.8)
- added SW3: SW_Push, Button_Switch_THT:SW_PUSH_6mm, F.Cu at (13.8, 16.0)
- added SW4: SW_Push, Button_Switch_THT:SW_PUSH_6mm, F.Cu at (13.8, 35.0)
- added SW5: SW_Push, Button_Switch_THT:SW_PUSH_6mm, F.Cu at (24.2, 25.5)
- added SW6: SW_Push, Button_Switch_THT:SW_PUSH_6mm, F.Cu at (21.8, -2.25)
- added SW7: SW_Push, Button_Switch_THT:SW_PUSH_6mm, F.Cu at (35.8, -2.25)
- added SW8: SW_Push, Button_Switch_THT:SW_PUSH_6mm, F.Cu at (49.8, -2.25)
- added SW9: SW_Push, Button_Switch_THT:SW_PUSH_6mm, F.Cu at (63.8, -2.25)
- added U1: ~, mux_breakout:MuxBreakout, F.Cu at (242.2, 118.8)
- A1: footprint Module:RaspberryPi_Pico_SMD_HandSolder -> Module:RaspberryPi_Pico_Common_THT
- moved A1 266.9 mm to (334.0, 30.0)
Connections:
- A1 pad 10: unconnected-(A1-GPIO7-Pad10) -> /AMUX_S1
- A1 pad 11: unconnected-(A1-GPIO8-Pad11) -> /JL_SEL
- A1 pad 12: unconnected-(A1-GPIO9-Pad12) -> /JR_SEL
- A1 pad 13: Net-(A1-GND-Pad13) -> GND
- A1 pad 14: unconnected-(A1-GPIO10-Pad14) -> /BTN_C
- A1 pad 15: unconnected-(A1-GPIO11-Pad15) -> /BTN_Z
- A1 pad 16: unconnected-(A1-GPIO12-Pad16) -> /BTN_LEFT
- A1 pad 17: unconnected-(A1-GPIO13-Pad17) -> /BTN_UP
- A1 pad 18: Net-(A1-GND-Pad13) -> GND
- A1 pad 19: unconnected-(A1-GPIO14-Pad19) -> /BTN_RIGHT
- A1 pad 20: unconnected-(A1-GPIO15-Pad20) -> /BTN_DOWN
- A1 pad 21: unconnected-(A1-GPIO16-Pad21) -> /BTN_LB
- A1 pad 22: unconnected-(A1-GPIO17-Pad22) -> /BTN_RB
- A1 pad 23: Net-(A1-GND-Pad13) -> GND
- A1 pad 24: unconnected-(A1-GPIO18-Pad24) -> /BTN_SEL
- A1 pad 25: unconnected-(A1-GPIO19-Pad25) -> /BTN_HOME
- A1 pad 26: unconnected-(A1-GPIO20-Pad26) -> /BTN_START
- A1 pad 27: unconnected-(A1-GPIO21-Pad27) -> /BTN_C
- A1 pad 28: Net-(A1-GND-Pad13) -> GND
- A1 pad 29: unconnected-(A1-GPIO22-Pad29) -> /BTN_Z
- A1 pad 3: Net-(A1-GND-Pad13) -> GND
- A1 pad 31: unconnected-(A1-GPIO26_ADC0-Pad31) -> /AMUX_SIG
- A1 pad 32: unconnected-(A1-GPIO27_ADC1-Pad32) -> /RGB_DIN
- A1 pad 33: unconnected-(A1-AGND-Pad33) -> GND
- A1 pad 36: unconnected-(A1-3V3-Pad36) -> +3V3
- A1 pad 38: Net-(A1-GND-Pad13) -> GND
- A1 pad 4: unconnected-(A1-GPIO2-Pad4) -> /BTN_X
- A1 pad 40: unconnected-(A1-VBUS-Pad40) -> +5V
- A1 pad 5: unconnected-(A1-GPIO3-Pad5) -> /BTN_Y
- A1 pad 6: unconnected-(A1-GPIO4-Pad6) -> /BTN_A
- A1 pad 7: unconnected-(A1-GPIO5-Pad7) -> /BTN_B
- A1 pad 8: Net-(A1-GND-Pad13) -> GND
- A1 pad 9: unconnected-(A1-GPIO6-Pad9) -> /AMUX_S0

Commit message: PCB WIP
Parts:
- moved A1 300.9 mm to (37.2, -19.3)
- moved U1 213.0 mm to (61.8, 5.50), turned to 90 degrees
- moved SW2 207.2 mm to (-6.25, -27.0)
- moved D4 166.3 mm to (110.5, -2.00)
- moved D1 162.7 mm to (99.8, 8.00)
- moved SW10 157.3 mm to (107.8, -27.0)
- moved D2 151.5 mm to (110.8, 18.0)
- moved D3 148.0 mm to (121.8, 8.00)
- moved SW7 38.6 mm to (49.8, 33.8)
- moved J2 36.0 mm to (98.0, 28.8)
- moved SW11 36.0 mm to (110.8, -11.5)
- moved SW12 36.0 mm to (110.8, 8.50)
- moved SW13 36.0 mm to (121.8, -1.50)
- moved SW14 36.0 mm to (119.8, 26.5)
- moved SW15 36.0 mm to (133.8, 16.5)
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Changed lines of the file:
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@@
 	(footprint "Button_Switch_THT:SW_PUSH_6mm"
 		(layer "F.Cu")
-		(at 85.75 -2.25)
+		(at 121.75 -1.5)
 		(descr "Generic 6mm SW tactile push button")
 		(tags "tact sw push 6mm")
@@
 	(footprint "Button_Switch_THT:SW_PUSH_6mm"
 		(layer "F.Cu")
-		(at 97.75 15.75)
+		(at 133.75 16.5)
 		(descr "Generic 6mm SW tactile push button")
 		(tags "tact sw push 6mm")
@@
 	(footprint "Button_Switch_THT:SW_PUSH-12mm"
 		(layer "F.Cu")
-		(at 173.6 75.825)
+		(at -6.25 -27)
 		(descr "Generic SW PUSH 12mm, e.g https://sten-eswitch-13110800-production.s3.amazonaws.com/system/asset/product_line/data_sheet/143/TL1100.pdf")
 		(tags "tact sw push 12mm")
@@
 	(footprint "Button_Switch_THT:SW_PUSH_6mm"
 		(layer "F.Cu")
-		(at 49.75 -2.25)
+		(at 85.75 -1.5)
 		(descr "Generic 6mm SW tactile push button")
 		(tags "tact sw push 6mm")
@@
 	(footprint "Button_Switch_THT:SW_PUSH_6mm"
 		(layer "F.Cu")
-		(at 63.75 -2.25)
+		(at 99.75 -1.5)
 		(descr "Generic 6mm SW tactile push button")
 		(tags "tact sw push 6mm")
@@
 	(footprint "adafruit_joystick_v2:JOYSTICK"
 		(layer "F.Cu")
-		(at 62 28)
+		(at 98 28.75)
 		(property "Reference" "J2"
 			(at -5.08 5.08 0)
@@
 	(footprint "Button_Switch_THT:SW_PUSH_6mm"
 		(layer "F.Cu")
-		(at 35.75 -2.25)
+		(at 49.75 33.75)
 		(descr "Generic 6mm SW tactile push button")
 		(tags "tact sw push 6mm")
@@
 	(footprint "Button_Switch_THT:SW_PUSH_6mm"
 		(layer "F.Cu")
-		(at 83.75 25.75)
+		(at 119.75 26.5)
 		(descr "Generic 6mm SW tactile push button")
 		(tags "tact sw push 6mm")
@@
 	(footprint "Module:RaspberryPi_Pico_Common_THT"
 		(layer "F.Cu")
-		(at 334 30)
+		(at 37.22 -19.32)
 		(descr "Raspberry Pi Pico common (Pico & Pico W) through-hole footprint, supports Raspberry Pi Pico 2, default socketed model has height of 8.51mm, https://datasheets.raspberrypi.com/pico/pico-datasheet.pdf")
 		(tags "module usb pcb antenna")
@@
 			(polygon
 				(pts
-					(xy 340.49 79.119895) (xy 335.79 75.469895) (xy 335.79 71.13) (xy 349.99 71.13) (xy 349.99 75.469895)
-					(xy 345.29 79.119895) (xy 345.29 80.13) (xy 340.49 80.13)
+					(xy 43.71 29.799895) (xy 39.01 26.149895) (xy 39.01 21.81) (xy 53.21 21.81) (xy 53.21 26.149895)
+					(xy 48.51 29.799895) (xy 48.51 30.81) (xy 43.71 30.81)
 				)
 			)
@@
 			(polygon
 				(pts
-					(xy 337.14 26.43) (xy 338.95 26.43) (xy 338.95 26.83) (xy 346.83 26.83) (xy 346.83 26.43) (xy 348.64 26.43)
-					(xy 348.64 6.93) (xy 337.14 6.93)
+					(xy 40.36 -22.89) (xy 42.17 -22.89) (xy 42.17 -22.49) (xy 50.05 -22.49) (xy 50.05 -22.89) (xy 51.86 -22.89)
+					(xy 51.86 -42.39) (xy 40.36 -42.39)
 				)
 			)
@@
 	(footprint "Button_Switch_THT:SW_PUSH-12mm"
 		(layer "F.Cu")
-		(at 190.3 106.925)
+		(at 107.75 -27)
 		(descr "Generic SW PUSH 12mm, e.g https://sten-eswitch-13110800-production.s3.amazonaws.com/system/asset/product_line/data_sheet/143/TL1100.pdf")
 		(tags "tact sw push 12mm")
@@
 	(footprint "Button_Switch_THT:SW_PUSH_6mm"
 		(layer "F.Cu")
-		(at 74.75 7.75)
+		(at 110.75 8.5)
 		(descr "Generic 6mm SW tactile push button")
 		(tags "tact sw push 6mm")
@@
 	(footprint "LED_THT:LED_D5.0mm-4_RGB_Wide_Pins"
 		(layer "F.Cu")
-		(at 254.345 81.425)
+		(at 110.5 -2)
 		(descr "LED, diameter 5.0mm, 4 pins, WP154A4, https://www.kingbright.com/attachments/file/psearch/000/00/00/L-154A4SUREQBFZGEW(Ver.11A).pdf")
 		(tags "LED diameter 5.0mm 2 pins diameter 5.0mm 3 pins diameter 5.0mm 4 pins RGB RGBLED")
@@
 	(footprint "Button_Switch_THT:SW_PUSH_6mm"
 		(layer "F.Cu")
-		(at 74.75 -12.25)
+		(at 110.75 -11.5)
 		(descr "Generic 6mm SW tactile push button")
 		(tags "tact sw push 6mm")
@@
 	(footprint "mux_breakout:MuxBreakout"
 		(layer "F.Cu")
-		(at 242.15 118.83)
+		(at 61.75 5.5 90)
 		(property "Reference" "U1"
-			(at 0 -5 0)
+			(at 0 -5 90)
 			(unlocked yes)
 			(layer "F.SilkS")
@@
 		)
 		(property "Value" "~"
-			(at 0 -3.5 0)
+			(at 0 -3.5 90)
 			(unlocked yes)
 			(layer "F.Fab")
@@
 		)
 		(property "Datasheet" ""
-			(at 0 0 0)
+			(at 0 0 90)
 			(unlocked yes)
 			(layer "F.Fab")
@@
 		)
 		(property "Description" "SparkFun CD74HC4067 breakout"
-			(at 0 0 0)
+			(at 0 0 90)
 			(unlocked yes)
 			(layer "F.Fab")
@@
 		)
 		(fp_text user "${REFERENCE}"
-			(at 0 -2 0)
+			(at 0 -2 90)
 			(unlocked yes)
 			(layer "F.Fab")
@@
 		)
 		(pad "1" thru_hole rect
-			(at -19.05 0)
+			(at -19.05 0 90)
 			(size 1.7 1.7)
 			(drill 1)
@@
 		)
 		(pad "2" thru_hole circle
-			(at -16.51 0)
+			(at -16.51 0 90)
 			(size 1.7 1.7)
 			(drill 1)
@@
 		)
 		(pad "3" thru_hole circle
-			(at -13.97 0)
+			(at -13.97 0 90)
 			(size 1.7 1.7)
 			(drill 1)
@@
 		)
 		(pad "4" thru_hole circle
-			(at -11.43 0)
+			(at -11.43 0 90)
 			(size 1.7 1.7)
 			(drill 1)
@@
 		)
 		(pad "5" thru_hole circle
-			(at -8.89 0)
+			(at -8.89 0 90)
 			(size 1.7 1.7)
 			(drill 1)
@@
 		)
 		(pad "6" thru_hole circle
-			(at -6.35 0)
+			(at -6.35 0 90)
 			(size 1.7 1.7)
 			(drill 1)
@@
 		)
 		(pad "7" thru_hole circle
-			(at -3.81 0)
+			(at -3.81 0 90)
 			(size 1.7 1.7)
 			(drill 1)
@@
 		)
 		(pad "8" thru_hole circle
-			(at -1.27 0)
+			(at -1.27 0 90)
 			(size 1.7 1.7)
 			(drill 1)
@@
 		)
 		(pad "9" thru_hole circle
-			(at 1.27 0)
+			(at 1.27 0 90)
 			(size 1.7 1.7)
 			(drill 1)
@@
 		)
 		(pad "10" thru_hole circle
-			(at 3.81 0)
+			(at 3.81 0 90)
 			(size 1.7 1.7)
 			(drill 1)
@@
 		)
 		(pad "11" thru_hole circle
-			(at 6.35 0)
+			(at 6.35 0 90)
 			(size 1.7 1.7)
 			(drill 1)
@@
 		)
 		(pad "12" thru_hole circle
-			(at 8.89 0)
+			(at 8.89 0 90)
 			(size 1.7 1.7)
 			(drill 1)
@@
 		)
 		(pad "13" thru_hole circle
-			(at 11.43 0)
+			(at 11.43 0 90)
 			(size 1.7 1.7)
 			(drill 1)
@@
 		)
 		(pad "14" thru_hole circle
-			(at 13.97 0)
+			(at 13.97 0 90)
 			(size 1.7 1.7)
 			(drill 1)
@@
 		)
 		(pad "15" thru_hole circle
-			(at 16.51 0)
+			(at 16.51 0 90)
 			(size 1.7 1.7)
 			(drill 1)
@@
 		)
 		(pad "16" thru_hole circle
-			(at 19.05 0)
+			(at 19.05 0 90)
 			(size 1.7 1.7)
 			(drill 1)
@@
 		)
 		(pad "17" thru_hole circle
-			(at 8.89 15.24)
+			(at 8.89 15.24 90)
 			(size 1.7 1.7)
 			(drill 1)
@@
 		)
 		(pad "18" thru_hole circle
-			(at 6.35 15.24)
+			(at 6.35 15.24 90)
 			(size 1.7 1.7)
 			(drill 1)
@@
 		)
 		(pad "19" thru_hole circle
-			(at 3.81 15.24)
+			(at 3.81 15.24 90)
 			(size 1.7 1.7)
 			(drill 1)
@@
 		)
 		(pad "20" thru_hole circle
-			(at 1.27 15.24)
+			(at 1.27 15.24 90)
 			(size 1.7 1.7)
 			(drill 1)
@@
 		)
 		(pad "21" thru_hole circle
-			(at -1.27 15.24)
+			(at -1.27 15.24 90)
 			(size 1.7 1.7)
 			(drill 1)
@@
 		)
 		(pad "22" thru_hole circle
-			(at -3.81 15.24)
+			(at -3.81 15.24 90)
 			(size 1.7 1.7)
 			(drill 1)
@@
 		)
 		(pad "23" thru_hole circle
-			(at -6.35 15.24)
+			(at -6.35 15.24 90)
 			(size 1.7 1.7)
 			(drill 1)
@@
 		)
 		(pad "24" thru_hole circle
-			(at -8.89 15.24)
+			(at -8.89 15.24 90)
 			(size 1.7 1.7)
 			(drill 1)
@@
 	(footprint "LED_THT:LED_D5.0mm-4_RGB_Wide_Pins"
 		(layer "F.Cu")
-		(at 254.345 73.875)
+		(at 121.76 8)
 		(descr "LED, diameter 5.0mm, 4 pins, WP154A4, https://www.kingbright.com/attachments/file/psearch/000/00/00/L-154A4SUREQBFZGEW(Ver.11A).pdf")
 		(tags "LED diameter 5.0mm 2 pins diameter 5.0mm 3 pins diameter 5.0mm 4 pins RGB RGBLED")
@@
 	(footprint "LED_THT:LED_D5.0mm-4_RGB_Wide_Pins"
 		(layer "F.Cu")
-		(at 254.345 58.775)
+		(at 99.76 8)
 		(descr "LED, diameter 5.0mm, 4 pins, WP154A4, https://www.kingbright.com/attachments/file/psearch/000/00/00/L-154A4SUREQBFZGEW(Ver.11A).pdf")
 		(tags "LED diameter 5.0mm 2 pins diameter 5.0mm 3 pins diameter 5.0mm 4 pins RGB RGBLED")
@@
 	(footprint "LED_THT:LED_D5.0mm-4_RGB_Wide_Pins"
 		(layer "F.Cu")
-		(at 254.345 66.325)
+		(at 110.76 18)
 		(descr "LED, diameter 5.0mm, 4 pins, WP154A4, https://www.kingbright.com/attachments/file/psearch/000/00/00/L-154A4SUREQBFZGEW(Ver.11A).pdf")
 		(tags "LED diameter 5.0mm 2 pins diameter 5.0mm 3 pins diameter 5.0mm 4 pins RGB RGBLED")
